File: Transformer/Transformer.kicad_sch (KiCad schematic)
At the start: 7 parts, among them J1 Conn_01x03, J2 Conn_01x02, T1 Transformer_SP_2S

Commit message: made dimensions multiples of 10 mm
Other:
- note added: "Consider adding fuse to this board"
Changed lines of the file:
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@@
     (stroke (width 0) (type default))
+  )
+  (text "Consider adding fuse to this board" (at 198.755 90.17 0)
+    (effects (font (size 1.27 1.27)) (justify left bottom))
   )
   (global_label "OUT2" (shape input) (at 151.765 97.155 0) (fields_autoplaced)
